Commit message: move the lidar behind a little

File: roomblock_description/robots/roomblock.urdf.xacro (robot description, xacro)
@@ -12,5 +12,5 @@
   </material>
   <joint name="block_joint" type="fixed">
-    <origin xyz="0 0 0.061" rpy="0 0 0" />
+    <origin xyz="-0.065 0 0.061" rpy="0 0 0" />
     <parent link="base_link"/>
     <child link="block_link" />
